Commit message: Moves camera link to line up more with camera in model.

File: traini_description/urdf/traini.urdf.xacro (robot description, xacro)
@@ -46,5 +46,5 @@
         <parent link="base_link"/>
         <child link="camera_link"/>
-        <origin xyz="0.1 0 0.3" rpy="0 0 0"/>
+        <origin xyz="0.1 0 0.055" rpy="0 0 0"/>
     </joint>
     <joint name="imu_joint" type="fixed">

Commit message: Moves indicator light to more reasonable spot and gives it's geometry a more reasonable size.

File: traini_description/urdf/traini.urdf.xacro (robot description, xacro)
@@ -30,5 +30,5 @@
         <visual name="indicator_light">
             <geometry>
-                <sphere radius="0.05"/>
+                <sphere radius="0.005"/>
             </geometry>
             <material name="indicator_light_material">
@@ -56,5 +56,5 @@
         <parent link="base_link"/>
         <child link="light_link"/>
-        <origin xyz="0 0 0.3" rpy="0 0 0"/>
+        <origin xyz="0 0 0.04" rpy="0 0 0"/>
     </joint>
 </robot>

Commit message: Adds optical frame for camera.

File: traini_description/urdf/traini.urdf.xacro (robot description, xacro)
@@ -21,4 +21,7 @@
     </link>
     <link name="camera_link">
+        <xacro:null_inertia/>
+    </link>
+    <link name="camera_link_optical">
         <xacro:null_inertia/>
     </link>
@@ -48,4 +51,9 @@
         <origin xyz="0.1 0 0.055" rpy="0 0 0"/>
     </joint>
+    <joint name="camera_joint_optical" type="fixed">
+        <parent link="camera_link"/>
+        <child link="camera_link_optical"/>
+        <origin xyz="0 0 0" rpy="-1.5707963 0.0 -1.5707963"/>
+    </joint>
     <joint name="imu_joint" type="fixed">
         <parent link="base_link"/>

Commit message: Tilts camera down

File: traini_description/urdf/traini.urdf.xacro (robot description, xacro)
@@ -49,5 +49,5 @@
         <parent link="base_link"/>
         <child link="camera_link"/>
-        <origin xyz="0.1 0 0.055" rpy="0 0 0"/>
+        <origin xyz="0.1 0 0.055" rpy="0 0.3 0"/>
     </joint>
     <joint name="camera_joint_optical" type="fixed">
